Commit message: gazebo ortamına aktarıldı kinematik ve hareket fonksiyonları yapılacak

File: workspace/src/my_robot_description/urdf/main.xacro (robot description, xacro)
@@ -1,5 +1,5 @@
 <?xml version="1.0"?>
 <robot name="my_robot" xmlns:xacro="http://www.ros.org/wiki/xacro">
+    <xacro:include filename="properties.xacro" />
     <xacro:include filename="my_robot.xacro" />
-    <xacro:include filename="properties.xacro" />
 </robot>

File: workspace/src/my_robot_description/urdf/my_robot.xacro (robot description, xacro)
@@ -1,11 +1,21 @@
 <?xml version="1.0"?>
 <robot name="my_robot" xmlns:xacro="http://www.ros.org/wiki/xacro">
+    <!-- Temel boyutlar -->
     <xacro:property name="base_width" value="0.6"/>
     <xacro:property name="base_length" value="0.4"/>
     <xacro:property name="base_height" value="0.2"/>
+    <!-- Tekerlek boyutları -->
     <xacro:property name="wheel_radius" value="0.1"/>
     <xacro:property name="wheel_length" value="0.05"/>
     <xacro:property name="caster_wheel_radius" value="0.05"/>
+    <!-- Hesaplanan yardımcı değişkenler (okunabilirlik için) -->
+    <xacro:property name="base_z" value="${(base_height/2) + wheel_radius}"/>
+    <xacro:property name="wheel_x" value="${-(base_width/2) + wheel_radius}"/>
+    <xacro:property name="wheel_y_offset" value="${(base_length/2) + (wheel_length/2)}"/>
+    <xacro:property name="wheel_z" value="${-wheel_radius}"/>
+    <xacro:property name="caster_z" value="${-((base_height/2) + caster_wheel_radius)}"/>
+    <!-- Base reference -->
     <link name="base_footprint"/>
+    <!-- Base gövdesi -->
     <link name="base_link">
         <visual>
@@ -13,8 +23,16 @@
                 <box size="${base_width} ${base_length} ${base_height}"/>
             </geometry>
-            <origin xyz="0.0 0.0 0.0" rpy="0.0 0.0 0.0"/>
+            <origin xyz="0 0 0" rpy="0 0 0"/>
             <material name="cyan"/>
         </visual>
+        <collision>
+            <geometry>
+                <box size="${base_width} ${base_length} ${base_height}"/>
+            </geometry>
+            <origin xyz="0 0 0" rpy="0 0 0"/>
+        </collision>
+        <xacro:box_inertia m="5.0" l="${base_length}" w="${base_width}" h="${base_height}" xyz="0 0 0" rpy="0 0 0"/>
     </link>
+    <!-- Tekerlek makrosu -->
     <xacro:macro name="wheel_link" params="prefix">
         <link name="${prefix}_wheel_link">
@@ -23,31 +41,46 @@
                     <cylinder radius="${wheel_radius}" length="${wheel_length}"/>
                 </geometry>
-                <origin xyz="0.0 0.0 0.0" rpy="${pi/2} 0.0 0.0"/>
+                <origin xyz="0 0 0" rpy="${pi/2} 0 0"/>
                 <material name="black"/>
             </visual>
+            <collision>
+                <geometry>
+                    <cylinder radius="${wheel_radius}" length="${wheel_length}"/>
+                </geometry>
+                <origin xyz="0 0 0" rpy="${pi/2} 0 0"/>
+            </collision>
+            <xacro:cylinder_inertia m="1.0" r="${wheel_radius}" h="${wheel_length}" xyz="0 0 0" rpy="${pi/2} 0 0"/>
         </link>
     </xacro:macro>
+    <!-- Tekerlek linkleri -->
     <xacro:wheel_link prefix="right"/>
     <xacro:wheel_link prefix="left"/>
+    <!-- Caster tekerlek -->
     <link name="caster_wheel_link">
-            <visual>
-                <geometry>
-                    <sphere radius="${caster_wheel_radius}"/>
-                </geometry>
-                <origin xyz="0.0 0.0 0.0" rpy="${pi/2} 0.0 0.0"/>
-                <material name="black"/>
-            </visual>
-        </link>
+        <visual>
+            <geometry>
+                <sphere radius="${caster_wheel_radius}"/>
+            </geometry>
+            <origin xyz="0 0 0" rpy="0 0 0"/>
+            <material name="black"/>
+        </visual>
+        <collision>
+            <geometry>
+                <sphere radius="${caster_wheel_radius}"/>
+            </geometry>
+            <origin xyz="0 0 0" rpy="0 0 0"/>
+        </collision>
+        <xacro:sphere_inertia m="0.5" r="${caster_wheel_radius}" xyz="0 0 0" rpy="0 0 0"/>
+    </link>
+    <!-- Eklem tanımları (hesaplanan property'leri kullanarak sadeleştirildi) -->
     <joint name="base_footprint_to_base_link" type="fixed">
         <parent link="base_footprint"/>
         <child link="base_link"/>
-        <origin xyz="0.0 0.0 ${(base_height/2) + wheel_radius}" rpy="0.0 0.0 0.0"/>
+        <origin xyz="0 0 ${base_z}" rpy="0 0 0"/>
     </joint>
     <joint name="base_right_wheel_joint" type="continuous">
         <parent link="base_link"/>
         <child link="right_wheel_link"/>
-        <origin xyz="${-(base_width/2) + (wheel_radius)}
-        ${-((base_length/2) + (wheel_length/2))}
-        ${-wheel_radius}" rpy="0.0 0.0 0.0"/>
+        <origin xyz="${wheel_x} ${-wheel_y_offset} ${wheel_z}" rpy="0 0 0"/>
         <axis xyz="0 1 0"/>
     </joint>
@@ -55,7 +88,5 @@
         <parent link="base_link"/>
         <child link="left_wheel_link"/>
-        <origin xyz="${-((base_width/2) - (wheel_radius))}
-        ${((base_length/2) + (wheel_length/2))}
-        ${-wheel_radius}" rpy="0.0 0.0 0.0"/>
+        <origin xyz="${wheel_x} ${wheel_y_offset} ${wheel_z}" rpy="0 0 0"/>
         <axis xyz="0 1 0"/>
     </joint>
@@ -63,5 +94,5 @@
         <parent link="base_link"/>
         <child link="caster_wheel_link"/>
-        <origin xyz="0.2 0.0 ${-((base_height/2) + caster_wheel_radius)}" rpy="0.0 0.0 0.0"/>
+        <origin xyz="0.2 0 ${caster_z}" rpy="0 0 0"/>
     </joint>
 </robot>

File: workspace/src/my_robot_description/urdf/properties.xacro (robot description, xacro)
@@ -7,3 +7,42 @@
         <color rgba="0.0 0.0 0.0 1.0"/>
     </material>
+    <xacro:macro name="box_inertia" params="m l w h xyz rpy">
+        <inertial>
+            <origin xyz="${xyz}" rpy="${rpy}"/>
+            <mass value="${m}"/>
+            <inertia
+                ixx="${(1/12.0) * m * (w*w + h*h)}"
+                ixy="0.0"
+                ixz="0.0"
+                iyy="${(1/12.0) * m * (l*l + h*h)}"
+                iyz="0.0"
+                izz="${(1/12.0) * m * (l*l + w*w)}"/>
+        </inertial>
+    </xacro:macro>
+    <xacro:macro name="cylinder_inertia" params="m r h xyz rpy">
+        <inertial>
+            <origin xyz="${xyz}" rpy="${rpy}"/>
+            <mass value="${m}"/>
+            <inertia
+                ixx="${(1/12.0) * m * (3*r*r + h*h)}"
+                ixy="0.0"
+                ixz="0.0"
+                iyy="${(1/12.0) * m * (3*r*r + h*h)}"
+                iyz="0.0"
+                izz="${(1/2.0) * m * r*r}"/>
+        </inertial>
+    </xacro:macro>
+    <xacro:macro name="sphere_inertia" params="m r xyz rpy">
+        <inertial>
+            <origin xyz="${xyz}" rpy="${rpy}"/>
+            <mass value="${m}"/>
+            <inertia
+                ixx="${(2/5.0) * m * r*r}"
+                ixy="0.0"
+                ixz="0.0"
+                iyy="${(2/5.0) * m * r*r}"
+                iyz="0.0"
+                izz="${(2/5.0) * m * r*r}"/>
+        </inertial>
+    </xacro:macro>
 </robot>

Commit message: gazeboo düzenlendi

File: workspace/src/my_robot_description/urdf/main.xacro (robot description, xacro)
@@ -1,6 +1,6 @@
-<?xml version="1.0"?>
-<robot name="my_robot" xmlns:xacro="http://www.ros.org/wiki/xacro">
-    <xacro:include filename="properties.xacro" />
-    <xacro:include filename="my_robot.xacro" />
-    <xacro:include filename="properties_gazebo.xacro" />
+<?xml version = "1.0"?>
+<robot name = "my_robot" xmlns:xacro="http://www.ros.org/wiki/xacro">
+    <xacro:include filename = "properties.xacro" />
+    <xacro:include filename = "properties_gazebo.xacro" />
+    <xacro:include filename = "my_robot.xacro" />
 </robot>

File: workspace/src/my_robot_description/urdf/my_robot.xacro (robot description, xacro)
@@ -1,98 +1,99 @@
-<?xml version="1.0"?>
-<robot name="my_robot" xmlns:xacro="http://www.ros.org/wiki/xacro">
-    <!-- Temel boyutlar -->
-    <xacro:property name="base_width" value="0.6"/>
-    <xacro:property name="base_length" value="0.4"/>
-    <xacro:property name="base_height" value="0.2"/>
-    <!-- Tekerlek boyutları -->
-    <xacro:property name="wheel_radius" value="0.1"/>
-    <xacro:property name="wheel_length" value="0.05"/>
-    <xacro:property name="caster_wheel_radius" value="0.05"/>
-    <!-- Hesaplanan yardımcı değişkenler (okunabilirlik için) -->
-    <xacro:property name="base_z" value="${(base_height/2) + wheel_radius}"/>
-    <xacro:property name="wheel_x" value="${-(base_width/2) + wheel_radius}"/>
-    <xacro:property name="wheel_y_offset" value="${(base_length/2) + (wheel_length/2)}"/>
-    <xacro:property name="wheel_z" value="${-wheel_radius}"/>
-    <xacro:property name="caster_z" value="${-((base_height/2) + caster_wheel_radius)}"/>
-    <!-- Base reference -->
-    <link name="base_footprint"/>
-    <!-- Base gövdesi -->
-    <link name="base_link">
+<?xml version = "1.0"?>
+<robot name = "my_robot" xmlns:xacro="http://www.ros.org/wiki/xacro">
+    <xacro:property name = "base_width" value = "0.6" />
+    <xacro:property name = "base_length" value = "0.4" />
+    <xacro:property name = "base_height" value = "0.2" />
+    <xacro:property name = "wheel_radius" value = "0.1" />
+    <xacro:property name = "wheel_length" value = "0.05" />
+    <xacro:property name = "caster_wheel_radius" value = "0.05" />
+    <xacro:macro name = "wheel_link" params = "prefix">
+        <link name = "${prefix}_wheel_link">
+            <visual>
+                <geometry>
+                    <cylinder radius = "${wheel_radius}" length = "${wheel_length}" />
+                </geometry>
+                <origin xyz = "0 0 0" rpy = "${pi/2} 0 0" />
+                <material name = "black" />
+            </visual>
+            <collision>
+                <geometry>
+                    <cylinder radius = "${wheel_radius}" length = "${wheel_length}" />
+                </geometry>
+                <origin xyz = "0 0 0" rpy = "${pi/2} 0 0" />
+            </collision>
+            <xacro:cylinder_inertia m = "1.0" r = "${2*wheel_radius}"
+                                              h = "${2*wheel_length}"
+                                              xyz = "0 0 0"
+                                              rpy = "${pi/2} 0 0" />
+        </link>
+    </xacro:macro>
+    <link name = "base_footprint" />
+    <link name = "base_link">
         <visual>
             <geometry>
-                <box size="${base_width} ${base_length} ${base_height}"/>
+                <box size = "${base_width} ${base_length} ${base_height}" />
             </geometry>
-            <origin xyz="0 0 0" rpy="0 0 0"/>
-            <material name="cyan"/>
+            <origin xyz = "0 0 0" rpy = "0 0 0" />
+            <material name = "cyan" />
         </visual>
         <collision>
             <geometry>
-                <box size="${base_width} ${base_length} ${base_height}"/>
+                <box size = "${base_width} ${base_length} ${base_height}" />
             </geometry>
-            <origin xyz="0 0 0" rpy="0 0 0"/>
+            <origin xyz = "0 0 0" rpy = "0 0 0" />
         </collision>
-        <xacro:box_inertia m="5.0" l="${2*base_length}" w="${2*base_width}" h="${2*base_height}" xyz="0 0 0" rpy="0 0 0"/>
+        <xacro:box_inertia m = "5.0" l = "${2*base_length}"
+                                     w = "${2*base_width}"
+                                     h = "${2*base_height}"
+                                     xyz = "0 0 0"
+                                     rpy = "0 0 0" />
     </link>
-    <!-- Tekerlek makrosu -->
-    <xacro:macro name="wheel_link" params="prefix">
-        <link name="${prefix}_wheel_link">
-            <visual>
-                <geometry>
-                    <cylinder radius="${wheel_radius}" length="${wheel_length}"/>
-                </geometry>
-                <origin xyz="0 0 0" rpy="${pi/2} 0 0"/>
-                <material name="black"/>
-            </visual>
-            <collision>
-                <geometry>
-                    <cylinder radius="${wheel_radius}" length="${wheel_length}"/>
-                </geometry>
-                <origin xyz="0 0 0" rpy="${pi/2} 0 0"/>
-            </collision>
-            <xacro:cylinder_inertia m="1.0" r="${2*wheel_radius}" h="${2*wheel_length}" xyz="0 0 0" rpy="${pi/2} 0 0"/>
-        </link>
-    </xacro:macro>
-    <!-- Tekerlek linkleri -->
-    <xacro:wheel_link prefix="right"/>
-    <xacro:wheel_link prefix="left"/>
-    <!-- Caster tekerlek -->
-    <link name="caster_wheel_link">
+    <xacro:wheel_link prefix = "right" />
+    <xacro:wheel_link prefix = "left" />
+    <link name = "caster_wheel_link">
         <visual>
             <geometry>
-                <sphere radius="${caster_wheel_radius}"/>
+                <sphere radius = "${caster_wheel_radius}" />
             </geometry>
-            <origin xyz="0 0 0" rpy="0 0 0"/>
-            <material name="black"/>
+            <origin xyz = "0 0 0" rpy = "0 0 0" />
+            <material name = "black" />
         </visual>
         <collision>
             <geometry>
-                <sphere radius="${caster_wheel_radius}"/>
+                <sphere radius = "${caster_wheel_radius}" />
             </geometry>
-            <origin xyz="0 0 0" rpy="0 0 0"/>
+            <origin xyz = "0 0 0" rpy = "0 0 0" />
         </collision>
-        <xacro:sphere_inertia m="0.5" r="${2*caster_wheel_radius}" xyz="0 0 0" rpy="0 0 0"/>
+        <xacro:sphere_inertia m = "0.5" r = "${2*caster_wheel_radius}"
+                                        xyz = "0 0 0"
+                                        rpy = "0 0 0" />
     </link>
-    <!-- Eklem tanımları (hesaplanan property'leri kullanarak sadeleştirildi) -->
-    <joint name="base_footprint_to_base_link" type="fixed">
-        <parent link="base_footprint"/>
-        <child link="base_link"/>
-        <origin xyz="0 0 ${base_z}" rpy="0 0 0"/>
+    <joint name = "base_joint" type = "fixed">
+        <parent link = "base_footprint" />
+        <child link  = "base_link" />
+        <origin xyz = "0 0 ${(base_height / 2) + wheel_radius}" rpy = "0 0 0" />
     </joint>
-    <joint name="base_right_wheel_joint" type="continuous">
-        <parent link="base_link"/>
-        <child link="right_wheel_link"/>
-        <origin xyz="${wheel_x} ${-wheel_y_offset} ${wheel_z}" rpy="0 0 0"/>
-        <axis xyz="0 1 0"/>
+    <joint name = "base_right_wheel_joint" type = "continuous">
+        <parent link = "base_link" />
+        <child link  = "right_wheel_link" />
+        <origin xyz = "${(-(base_width / 2)) + wheel_radius}
+                       ${-((base_length / 2) + (wheel_length / 2))}
+                       ${-wheel_radius}"
+                       rpy = "0 0 0" />
+        <axis xyz = "0 1 0" />
     </joint>
-    <joint name="base_left_wheel_joint" type="continuous">
-        <parent link="base_link"/>
-        <child link="left_wheel_link"/>
-        <origin xyz="${wheel_x} ${wheel_y_offset} ${wheel_z}" rpy="0 0 0"/>
-        <axis xyz="0 1 0"/>
+    <joint name = "base_left_wheel_joint" type = "continuous">
+        <parent link = "base_link" />
+        <child link  = "left_wheel_link" />
+        <origin xyz = "${(-(base_width / 2)) + wheel_radius}
+                       ${(base_length / 2) + (wheel_length / 2)}
+                       ${-wheel_radius}"
+                       rpy = "0 0 0" />
+        <axis xyz = "0 1 0" />
     </joint>
-    <joint name="base_caster_wheel_joint" type="fixed">
-        <parent link="base_link"/>
-        <child link="caster_wheel_link"/>
-        <origin xyz="0.2 0 ${caster_z}" rpy="0 0 0"/>
+    <joint name = "base_caster_wheel_joint" type = "fixed">
+        <parent link = "base_link" />
+        <child link  = "caster_wheel_link" />
+        <origin xyz = "0.2 0 ${-((base_height / 2) + caster_wheel_radius)}" rpy = "0 0 0" />
     </joint>
 </robot>

File: workspace/src/my_robot_description/urdf/properties.xacro (robot description, xacro)
@@ -1,47 +1,35 @@
-<?xml version="1.0"?>
-<robot name="my_robot" xmlns:xacro="http://www.ros.org/wiki/xacro">
-    <material name="cyan">
-        <color rgba="0.0 1.0 1.0 1"/>
+<?xml version = "1.0"?>
+<robot name = "my_robot" xmlns:xacro="http://www.ros.org/wiki/xacro">
+    <material name = "cyan">
+        <color rgba = "0 1 1 1" />
     </material>
-    <material name="black">
-        <color rgba="0.0 0.0 0.0 1.0"/>
+    <material name = "black">
+        <color rgba = "0 0 0 1" />
     </material>
-    <xacro:macro name="box_inertia" params="m l w h xyz rpy">
+    <xacro:macro name = "box_inertia" params = "m l w h xyz rpy">
         <inertial>
-            <origin xyz="${xyz}" rpy="${rpy}"/>
-            <mass value="${m}"/>
-            <inertia
-                ixx="${(1/12.0) * m * (w*w + h*h)}"
-                ixy="0.0"
-                ixz="0.0"
-                iyy="${(1/12.0) * m * (l*l + h*h)}"
-                iyz="0.0"
-                izz="${(1/12.0) * m * (l*l + w*w)}"/>
+            <origin xyz = "${xyz}" rpy = "${rpy}" />
+            <mass value = "${m}" />
+            <inertia ixx = "${(m / 12) * (h*h + l*l)}" ixy = "0" ixz = "0"
+                     iyy = "${(m / 12) * (w*w + l*l)}" iyz = "0"
+                     izz = "${(m / 12) * (w*w + h*h)}" />
         </inertial>
     </xacro:macro>
-    <xacro:macro name="cylinder_inertia" params="m r h xyz rpy">
+    <xacro:macro name = "cylinder_inertia" params = "m r h xyz rpy">
         <inertial>
-            <origin xyz="${xyz}" rpy="${rpy}"/>
-            <mass value="${m}"/>
-            <inertia
-                ixx="${(1/12.0) * m * (3*r*r + h*h)}"
-                ixy="0.0"
-                ixz="0.0"
-                iyy="${(1/12.0) * m * (3*r*r + h*h)}"
-                iyz="0.0"
-                izz="${(1/2.0) * m * r*r}"/>
+            <origin xyz = "${xyz}" rpy = "${rpy}" />
+            <mass value = "${m}" />
+            <inertia ixx = "${(m / 12) * (3*r*r + h*h)}" ixy = "0" ixz = "0"
+                     iyy = "${(m / 12) * (3*r*r + h*h)}" iyz = "0"
+                     izz = "${(m / 2)  * (r*r)}" />
         </inertial>
     </xacro:macro>
-    <xacro:macro name="sphere_inertia" params="m r xyz rpy">
+    <xacro:macro name = "sphere_inertia" params = "m r xyz rpy">
         <inertial>
-            <origin xyz="${xyz}" rpy="${rpy}"/>
-            <mass value="${m}"/>
-            <inertia
-                ixx="${(2/5.0) * m * r*r}"
-                ixy="0.0"
-                ixz="0.0"
-                iyy="${(2/5.0) * m * r*r}"
-                iyz="0.0"
-                izz="${(2/5.0) * m * r*r}"/>
+            <origin xyz = "${xyz}" rpy = "${rpy}" />
+            <mass value = "${m}" />
+            <inertia ixx = "${(2 / 5) * m * r * r}" ixy = "0" ixz = "0"
+                     iyy = "${(2 / 5) * m * r * r}" iyz = "0"
+                     izz = "${(2 / 5) * m * r * r}" />
         </inertial>
     </xacro:macro>

File: workspace/src/my_robot_description/urdf/properties_gazebo.xacro (robot description, xacro)
@@ -1,17 +1,36 @@
-<?xml version="1.0"?>
-<robot name="my_robot" xmlns:xacro="http://www.ros.org/wiki/xacro">
-    <gazebo reference="base_link">
-        <mu1>1.0</mu1>
-        <mu2>1.0</mu2>
+<?xml version = "1.0"?>
+<robot name = "my_robot" xmlns:xacro="http://www.ros.org/wiki/xacro">
+    <gazebo reference = "base_link">
         <material>Gazebo/Blue</material>
     </gazebo>
-    <gazebo reference="left_wheel_link">
+    <gazebo reference = "right_wheel_link">
         <material>Gazebo/Black</material>
     </gazebo>
-    <gazebo reference="right_wheel_link">
+    <gazebo reference = "left_wheel_link">
         <material>Gazebo/Black</material>
     </gazebo>
-    <gazebo reference="caster_wheel_link">
-        <material>Gazebo/Gray</material>
+    <gazebo reference = "caster_wheel_link">
+        <material>Gazebo/Black</material>
+        <mu1 value = "0.1" />
+        <mu2 value = "0.1" />
+    </gazebo>
+    <gazebo>
+        <plugin name="diff_drive_controller" filename="libgazebo_ros_diff_drive.so">
+        <!-- Update rate in Hz -->
+        <update_rate>50</update_rate>
+        <!-- wheels -->
+        <left_joint>base_left_wheel_joint</left_joint>
+        <right_joint>base_right_wheel_joint</right_joint>
+        <!-- kinematics -->
+        <wheel_separation>0.45</wheel_separation>
+        <wheel_diameter>0.2</wheel_diameter>
+        <!-- output -->
+        <publish_odom>true</publish_odom>
+        <publish_odom_tf>true</publish_odom_tf>
+        <publish_wheel_tf>true</publish_wheel_tf>
+        <odometry_topic>odom</odometry_topic>
+        <odometry_frame>odom</odometry_frame>
+        <robot_base_frame>base_footprint</robot_base_frame>
+        </plugin>
     </gazebo>
 </robot>
